File: IMU_Schematic/IMU_Schematic.kicad_sch (KiCad schematic)
At the start: 0 parts

Commit message: Added Gyro and Teensy libraries
Parts:
- added U1: IAM-20380, IAM-20380_IVS, symbol 2025-10-22_23-56-09:IAM-20380
- added U2: DEV-16771, DEV-16771:MODULE_DEV-16771, symbol DEV-16771:DEV-16771
